File: S3_stamp.kicad_sch (KiCad schematic)
At the start: 39 parts, among them J1 Conn_South, J2 Conn_North, J3 Conn_East, J4 Conn_West, Q1 BSS84, SW2 SW_RESET, U2 AP2112K-3.3, U4 MCP73831, U5 ESP32-S3, U6 W25Q16JVSSIQ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

Commit message: update and 3D models
Parts:
- added JP3: Jumper_Neopixel_VDD, Jumper:SolderJumper-2_P1.3mm_Bridged_RoundedPad1.0x1.5mm, symbol Jumper:Jumper_2_Bridged
Connections:
- net GPIO21: now also JP3.2 (B); no longer D3.3 (DIN)
- new net: D3.3 (DIN), JP3.1 (A)
Other:
- moved on the sheet: D3, JP1
Changed lines of the file:
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@@
 	)
 	(no_connect
-		(at 113.03 170.18)
+		(at 119.38 135.89)
 	)
 	(no_connect
@@
 	(wire
 		(pts
-			(xy 96.52 172.72) (xy 96.52 173.99)
+			(xy 102.87 138.43) (xy 102.87 139.7)
 		)
 		(stroke
@@
 	(wire
 		(pts
-			(xy 97.79 172.72) (xy 96.52 172.72)
+			(xy 104.14 138.43) (xy 102.87 138.43)
 		)
 		(stroke
@@
 	(wire
 		(pts
+			(xy 102.87 135.89) (xy 104.14 135.89)
+		)
+		(stroke
+			(width 0)
+			(type solid)
+		)
+	)
+	(wire
+		(pts
 			(xy 115.57 95.25) (xy 115.57 92.71)
 		)
@@
 	(wire
 		(pts
-			(xy 85.09 170.18) (xy 97.79 170.18)
+			(xy 91.44 135.89) (xy 92.71 135.89)
 		)
 		(stroke
@@
 	(wire
 		(pts
-			(xy 96.52 166.37) (xy 96.52 167.64)
+			(xy 102.87 132.08) (xy 102.87 133.35)
 		)
 		(stroke
@@
 	(wire
 		(pts
-			(xy 97.79 167.64) (xy 96.52 167.64)
+			(xy 104.14 133.35) (xy 102.87 133.35)
 		)
 		(stroke
@@
 	(wire
 		(pts
-			(xy 96.52 154.94) (xy 96.52 156.21)
+			(xy 102.87 120.65) (xy 102.87 121.92)
 		)
 		(stroke
@@
 		)
 	)
-	(label "GPIO21"
-		(at 85.09 170.18 180)
-		(fields_autoplaced yes)
-		(effects
-			(font
-				(size 1.27 1.27)
-			)
-			(justify right bottom)
-		)
-	)
 	(global_label "GPIO0{slash}BOOT"
 		(shape input)
@@
 		)
 	)
+	(global_label "GPIO21"
+		(shape input)
+		(at 91.44 135.89 180)
+		(fields_autoplaced yes)
+		(effects
+			(font
+				(size 1.27 1.27)
+			)
+			(justify right)
+		)
+		(property "Intersheetrefs" "${INTERSHEET_REFS}"
+			(at 81.5605 135.89 0)
+			(effects
+				(font
+					(size 1.27 1.27)
+				)
+				(justify right)
+				(hide yes)
+			)
+		)
+	)
 	(global_label "GPIO38"
 		(shape input)
@@
 	(symbol
 		(lib_id "power:+3.3V")
-		(at 96.52 154.94 0)
+		(at 102.87 120.65 0)
 		(mirror y)
 		(unit 1)
@@
 		(dnp no)
 		(property "Reference" "#PWR0137"
-			(at 96.52 158.75 0)
+			(at 102.87 124.46 0)
 			(effects
 				(font
@@
 		)
 		(property "Value" "+3V3"
-			(at 96.52 151.13 0)
+			(at 102.87 116.84 0)
 			(effects
 				(font
@@
 		)
 		(property "Footprint" ""
-			(at 96.52 154.94 0)
+			(at 102.87 120.65 0)
 			(effects
 				(font
@@
 		)
 		(property "Datasheet" ""
-			(at 96.52 154.94 0)
+			(at 102.87 120.65 0)
 			(effects
 				(font
@@
 		)
 		(property "Description" ""
-			(at 96.52 154.94 0)
+			(at 102.87 120.65 0)
 			(effects
 				(font
@@
 	)
 	(symbol
+		(lib_id "Jumper:Jumper_2_Bridged")
+		(at 97.79 135.89 0)
+		(mirror y)
+		(unit 1)
+		(exclude_from_sim no)
+		(in_bom yes)
+		(on_board yes)
+		(dnp no)
+		(property "Reference" "JP3"
+			(at 98.4249 140.97 90)
+			(effects
+				(font
+					(size 1.27 1.27)
+				)
+				(justify left)
+			)
+		)
+		(property "Value" "Jumper_Neopixel_VDD"
+			(at 97.79 133.35 0)
+			(effects
+				(font
+					(size 1.27 1.27)
+				)
+				(hide yes)
+			)
+		)
+		(property "Footprint" "Jumper:SolderJumper-2_P1.3mm_Bridged_RoundedPad1.0x1.5mm"
+			(at 97.79 135.89 0)
+			(effects
+				(font
+					(size 1.27 1.27)
+				)
+				(hide yes)
+			)
+		)
+		(property "Datasheet" "~"
+			(at 97.79 135.89 0)
+			(effects
+				(font
+					(size 1.27 1.27)
+				)
+				(hide yes)
+			)
+		)
+		(property "Description" ""
+			(at 97.79 135.89 0)
+			(effects
+				(font
+					(size 1.27 1.27)
+				)
+				(hide yes)
+			)
+		)
+		(pin "1"
+		)
+		(pin "2"
+		)
+		(instances
+			(project "S3_stamp"
+				(path "/872e912f-cc14-4edf-9f9a-f509de06f155"
+					(reference "JP3")
+					(unit 1)
+				)
+			)
+		)
+	)
+	(symbol
 		(lib_id "Battery_Management_Extra:MCP73831")
 		(at 58.42 91.44 0)
@@
 	(symbol
 		(lib_id "Jumper:Jumper_2_Bridged")
-		(at 96.52 161.29 270)
+		(at 102.87 127 270)
 		(mirror x)
 		(unit 1)
@@
 		(dnp no)
 		(property "Reference" "JP1"
-			(at 91.44 161.9249 90)
+			(at 97.79 127.6349 90)
 			(effects
 				(font
@@
 		)
 		(property "Value" "Jumper_Neopixel_VDD"
-			(at 99.06 161.29 0)
+			(at 105.41 127 0)
 			(effects
 				(font
@@
 		)
 		(property "Footprint" "Jumper:SolderJumper-2_P1.3mm_Bridged_RoundedPad1.0x1.5mm"
-			(at 96.52 161.29 0)
+			(at 102.87 127 0)
 			(effects
 				(font
@@
 		)
 		(property "Datasheet" "~"
-			(at 96.52 161.29 0)
+			(at 102.87 127 0)
 			(effects
 				(font
@@
 		)
 		(property "Description" ""
-			(at 96.52 161.29 0)
+			(at 102.87 127 0)
 			(effects
 				(font
@@
 	(symbol
 		(lib_id "power:GND")
-		(at 96.52 173.99 0)
+		(at 102.87 139.7 0)
 		(unit 1)
 		(exclude_from_sim no)
@@
 		(dnp no)
 		(property "Reference" "#PWR0115"
-			(at 96.52 180.34 0)
+			(at 102.87 146.05 0)
 			(effects
 				(font
@@
 		)
 		(property "Value" "GND"
-			(at 96.52 177.8 0)
+			(at 102.87 143.51 0)
 			(effects
 				(font
@@
 		)
 		(property "Footprint" ""
-			(at 96.52 173.99 0)
+			(at 102.87 139.7 0)
 			(effects
 				(font
@@
 		)
 		(property "Datasheet" ""
-			(at 96.52 173.99 0)
+			(at 102.87 139.7 0)
 			(effects
 				(font
@@
 		)
 		(property "Description" ""
-			(at 96.52 173.99 0)
+			(at 102.87 139.7 0)
 			(effects
 				(font
@@
 	(symbol
 		(lib_id "LED_Extra:WS2812B-2020")
-		(at 105.41 170.18 0)
+		(at 111.76 135.89 0)
 		(unit 1)
 		(exclude_from_sim no)
@@
 		(dnp no)
 		(property "Reference" "D3"
-			(at 109.22 163.83 0)
+			(at 115.57 129.54 0)
 			(effects
 				(font
@@
 		)
 		(property "Value" "WS2812B-2020"
-			(at 106.68 176.53 0)
+			(at 113.03 142.24 0)
 			(effects
 				(font
@@
 		)
 		(property "Footprint" "LED_SMD:LED_WS2812B-2020_PLCC4_2.0x2.0mm"
-			(at 106.68 177.8 0)
+			(at 113.03 143.51 0)
 			(effects
 				(font
@@
 		)
 		(property "Datasheet" "https://www.tme.eu/Document/4a8239e52df5e0b5cc2eb96834c5d8b6/WS2812B-2020.pdf"
-			(at 107.95 179.705 0)
+			(at 114.3 145.415 0)
 			(effects
 				(font
@@
 		)
 		(property "Description" ""
-			(at 105.41 170.18 0)
+			(at 111.76 135.89 0)
 			(effects
 				(font
@@
 		)
 		(property "LCSC" "C965555"
-			(at 105.41 170.18 0)
+			(at 111.76 135.89 0)
 			(effects
 				(font

Commit message: further development
Parts:
- J1, J2, J3, J4: footprint RP2040_stamp:Castellated_1x10_P2.00mm_Vertical -> Connector_PinHeader_2.00mm:PinHeader_1x10_P2.00mm_Vertical
Changed lines of the file:
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@@
 		)
 		(property "Value" "Conn_West"
-			(at 231.648 87.63 90)
-			(effects
-				(font
-					(size 1.27 1.27)
-				)
-			)
-		)
-		(property "Footprint" "RP2040_stamp:Castellated_1x10_P2.00mm_Vertical"
+			(at 221.488 107.442 0)
+			(effects
+				(font
+					(size 1.27 1.27)
+				)
+			)
+		)
+		(property "Footprint" "Connector_PinHeader_2.00mm:PinHeader_1x10_P2.00mm_Vertical"
 			(at 228.6 87.63 0)
 			(effects
@@
 		)
 		(property "Value" "Conn_North"
-			(at 241.3 77.978 90)
-			(effects
-				(font
-					(size 1.27 1.27)
-				)
-			)
-		)
-		(property "Footprint" "RP2040_stamp:Castellated_1x10_P2.00mm_Vertical"
+			(at 224.79 64.008 90)
+			(effects
+				(font
+					(size 1.27 1.27)
+				)
+			)
+		)
+		(property "Footprint" "Connector_PinHeader_2.00mm:PinHeader_1x10_P2.00mm_Vertical"
 			(at 241.3 74.93 0)
 			(effects
@@
 		)
 		(property "Value" "Conn_East"
-			(at 253.492 87.63 90)
-			(effects
-				(font
-					(size 1.27 1.27)
-				)
-			)
-		)
-		(property "Footprint" "RP2040_stamp:Castellated_1x10_P2.00mm_Vertical"
+			(at 261.874 103.886 0)
+			(effects
+				(font
+					(size 1.27 1.27)
+				)
+			)
+		)
+		(property "Footprint" "Connector_PinHeader_2.00mm:PinHeader_1x10_P2.00mm_Vertical"
 			(at 256.54 87.63 0)
 			(effects
@@
 		)
 		(property "Value" "Conn_South"
-			(at 241.3 99.822 90)
-			(effects
-				(font
-					(size 1.27 1.27)
-				)
-			)
-		)
-		(property "Footprint" "RP2040_stamp:Castellated_1x10_P2.00mm_Vertical"
+			(at 242.316 119.888 90)
+			(effects
+				(font
+					(size 1.27 1.27)
+				)
+			)
+		)
+		(property "Footprint" "Connector_PinHeader_2.00mm:PinHeader_1x10_P2.00mm_Vertical"
 			(at 241.3 102.87 0)
 			(effects
