File: S3_stamp.kicad_pcb (KiCad board)
At the start: 4 copper layers, 25 x 25 mm, 39 parts, among them J1 Conn_South, J2 Conn_North, J3 Conn_East, J4 Conn_West, Q1 BSS84, SW2 SW_RESET, U2 AP2112K-3.3, U4 MCP73831, U5 ESP32-S3, U6 W25Q16JVSSIQ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

Commit message: update and 3D models
Parts:
- added JP3: Jumper_Neopixel_VDD, Jumper:SolderJumper-2_P1.3mm_Bridged_RoundedPad1.0x1.5mm, B.Cu at (155.3, 114.0)
- moved JP1 0.90 mm to (155.3, 112.7)
- moved C14 0.49 mm to (148.2, 102.0)
- moved C23 0.37 mm to (147.8, 103.5)
- moved C17 0.35 mm to (148.7, 103.5)
- moved JP2 0.16 mm to (159.8, 114.3)
- moved C21 0.05 mm to (152.0, 103.5)
Connections:
- D3 pad 3: GPIO21 -> Net-(D3-DIN)
Routing:
- net Net-(D3-DIN): track 0.00 -> 4.14 mm, vias 0 -> 1
- net GND: track 5.09 -> 3.18 mm
- net VDD_SPI: track 12.5 -> 13.8 mm
- net Net-(D3-VDD): track 0.80 -> 1.67 mm
- net +3V3: track 31.5 -> 30.6 mm
- net GPIO21: track 10.8 -> 11.6 mm, vias 0 -> 1
- net Net-(U5-XTAL_P): track 6.82 -> 7.46 mm
Other:
- board text added: "48"
- board text added: "neop 3,3V"
- board text added: "neop IO21"
- board text removed: "G"

Commit message: further development
Parts:
- J1, J2, J3, J4: footprint RP2040_stamp:Castellated_1x10_P2.00mm_Vertical -> Connector_PinHeader_2.00mm:PinHeader_1x10_P2.00mm_Vertical
- moved C4 18.2 mm to (157.2, 99.5)
- moved C18 0.45 mm to (160.0, 99.8)
- moved C16 0.40 mm to (160.1, 105.1)
- moved U4 0.40 mm to (159.6, 102.3)
- moved D2 0.25 mm to (157.2, 103.7)
- moved R7 0.25 mm to (157.2, 101.8)
- moved U5 0.23 mm to (150.4, 109.0)
- moved R8 0.10 mm to (157.6, 105.4)
- moved D1 0.10 mm to (156.4, 97.2)
Routing:
- net +3V3: track 30.6 -> 33.3 mm
- net GPIO0/BOOT: track 20.2 -> 22.5 mm
- net VBAT: track 9.72 -> 11.9 mm
- net GPIO48: track 18.1 -> 20.3 mm
- net +5V: track 17.9 -> 20.0 mm
- net GPIO47: track 17.6 -> 19.6 mm
- net USB_D+: track 19.1 -> 21.1 mm
- net USB_D-: track 20.6 -> 22.1 mm
- net RESET: track 29.3 -> 30.8 mm
- net GPIO33: track 14.3 -> 15.8 mm
- net MTCK: track 15.3 -> 16.7 mm
- net GPIO46: track 15.7 -> 17.1 mm
- net GPIO45: track 14.5 -> 15.9 mm
- net GPIO38: track 14.9 -> 16.0 mm
- net GPIO11: track 6.19 -> 7.09 mm
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Other:
- board text added: "50Ω"
- board text added: "BATT 500mA CHG"
- board text added: "CERN OHL-P"
- board text added: "ESP32-S3"
- board text added: "IO21"
- board text added: "RST"
- board text added: "stamp"
- board text removed: "BATT"

Commit message: new picture and gerbers
Routing:
- net Net-(D3-DIN): track 4.14 -> 2.43 mm
- net +3V3: track 33.3 -> 32.3 mm
Other:
- board text added: "2MB 8MB 16MB"
- board text added: "4MB 8MB 16MB"
- board text added: "RAM"
- board text added: "flash"
